File: CANGatewayE.kicad_pcb (KiCad board)
At the start: 4 copper layers, 49.8 x 25.4 mm, 67 parts, among them J1 RJ45_Amphenol_RJMG1BD3B8K1ANR, J3 Conn_01x10, J4 Conn_01x10, SW1 SW_DIP_x02, U1 STM32H563RGTx, U2 LAN8742A, U3 MCP2562-E-SN, U4 MCP2562-E-SN, U5 ME6119A33PG, U7 ME6210A50PG, Y1 24MHz, Y2 25MHz

Commit message: fix
Parts:
- removed J1: RJ45_Amphenol_RJMG1BD3B8K1ANR, Connector_RJ:RJ45_Amphenol_RJMG1BD3B8K1ANR
- added J5: RJ45_Hanrun_HR911105A_Horizontal, Connector_RJ:RJ45_Hanrun_HR911105A_Horizontal, F.Cu at (118.1, 84.5)
- added R23: 10k, Resistor_SMD:R_0402_1005Metric, F.Cu at (124.3, 97.6)
- added TP1: TestPoint, TestPoint:TestPoint_Pad_D1.0mm, B.Cu at (136.4, 80.8)
- added TP2: TestPoint, TestPoint:TestPoint_Pad_D1.0mm, B.Cu at (138.7, 80.8)
- R12, R13, R14, R15, R19, R20: moved to F.Cu
- U3, U4: value MCP2562-E-SN -> MCP2562FD-E-SN
- moved R20 18.3 mm to (148.3, 79.2), turned to 180 degrees
- moved R19 15.5 mm to (148.1, 95.8), turned to 180 degrees
- moved U3 8.13 mm to (148.3, 93.0), turned to -90 degrees
- moved U4 8.13 mm to (148.3, 84.8), turned to 90 degrees
- moved JP2 5.47 mm to (147.3, 86.9)
- moved JP3 5.47 mm to (149.4, 86.9)
- moved JP4 5.47 mm to (149.4, 81.8)
- moved JP5 5.47 mm to (147.3, 81.8)
- moved D1 2.03 mm to (119.9, 79.2)
- moved D2 2.03 mm to (119.9, 77.2)
- moved R21 2.03 mm to (122.9, 79.2)
- moved R22 2.03 mm to (122.9, 77.4)
- moved R13 0.80 mm to (124.2, 86.6)
- moved R15 0.57 mm to (123.7, 89.9), turned to -90 degrees
- moved R14 0.57 mm to (124.2, 91.9)
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Connections:
- J3 pad 1: GND -> /SPI3_MOSI
- J3 pad 10: /CAN/CAN2_H -> /CAN/CAN1_H
- J3 pad 2: unconnected-(J3-Pin_2-Pad2) -> /SPI3_MISO
- J3 pad 3: unconnected-(J3-Pin_3-Pad3) -> /SPI3_SCK
- J3 pad 4: unconnected-(J3-Pin_4-Pad4) -> /SPI3_CS
- J3 pad 5: /Connector/VCP_TX -> /VCP_TX
- J3 pad 6: /Connector/VCP_RX -> /VCP_RX
- J3 pad 7: /CAN2_RD -> /CAN1_RD
- J3 pad 8: /CAN2_TD -> /CAN1_TD
- J3 pad 9: /CAN/CAN2_L -> /CAN/CAN1_L
- J4 pad 10: /CAN/CAN1_H -> /CAN/CAN2_H
- J4 pad 7: /CAN1_RD -> /CAN2_RD
- J4 pad 8: /CAN1_TD -> /CAN2_TD
- J4 pad 9: /CAN/CAN1_L -> /CAN/CAN2_L
- R21 pad 1: /MCU/PB15 -> /MCU/PC7
- R22 pad 1: /MCU/PB14 -> /MCU/PC8
- SW1 pad 1: /CAN/CAN1_L -> /CAN/CAN2_L
- SW1 pad 2: Net-(R20-Pad2) -> Net-(R19-Pad1)
- SW1 pad 3: /CAN/CAN2_L -> /CAN/CAN1_L
- SW1 pad 4: Net-(R19-Pad1) -> Net-(R20-Pad2)
- U1 pad 10: /MCU/PC2 -> /SPI3_MISO
- U1 pad 11: /MCU/PC3 -> /SPI3_MOSI
- U1 pad 17: /MCU/PA3 -> /SPI3_CS
- U1 pad 34: /RMII_TXD1 -> /MCU/PB13
- U1 pad 36: /MCU/PB15 -> /RMII_TXD1
- U1 pad 42: /MCU/PA9 -> /SPI3_SCK
- U1 pad 43: /CAN2_TD -> /MCU/PA10
- U1 pad 44: /CAN1_RD -> /MCU/PA11
- U1 pad 45: /CAN1_TD -> /MCU/PA12
- U1 pad 51: /MCU/PC10 -> /VCP_TX
- U1 pad 52: /MCU/PC11 -> /VCP_RX
- U1 pad 58: /MCU/PB6 -> /CAN2_TD
- U1 pad 59: /MCU/PB7 -> /CAN1_TD
- U1 pad 61: /MCU/PB8 -> /CAN1_RD
Routing:
- net /SPI3_SCK: track 0.00 -> 26.0 mm, vias 0 -> 2
- net /VCP_TX: track 0.00 -> 19.8 mm, vias 0 -> 1
- net /VCP_RX: track 0.00 -> 17.4 mm, vias 0 -> 1
- net /MCU/PC8: track 0.00 -> 16.0 mm, vias 0 -> 2
- net /MCU/PC7: track 0.00 -> 14.6 mm, vias 0 -> 2
- net /MCU/PB15: track 14.5 -> 0.00 mm, vias 2 -> 0
- net /MCU/PB14: track 13.0 -> 0.00 mm, vias 2 -> 0
- net /SPI3_MOSI: track 0.00 -> 12.2 mm
- net /SPI3_MISO: track 0.00 -> 10.9 mm
- net /CAN2_TD: track 29.1 -> 18.8 mm, vias 2 -> 1
- net /SPI3_CS: track 0.00 -> 9.11 mm, vias 0 -> 1
- net /CAN1_RD: track 14.0 -> 21.0 mm
- net /Ethernet/LED2: track 30.5 -> 37.4 mm, vias 2 -> 3
- net /CAN/CAN2_L: track 10.0 -> 15.8 mm
- net /CAN/CAN1_L: track 15.9 -> 10.6 mm
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Other:
- board size 49.8 x 25.4 mm -> 46.6 x 25.4 mm
- board text removed: "CAN1"
- board text removed: "CAN2"
