File: CANGatewayE.kicad_sch (KiCad schematic)
At the start: 4 parts

Commit message: fix
Parts:
- added TP1, TP2: TestPoint, TestPoint:TestPoint_Pad_D1.0mm, symbol Connector:TestPoint
Connections:
- net MCU/PB15 is gone; now on net MCU/PC7: R21.1
- net MCU/PB14: no longer R22.1
- net MCU/PC8: now also R22.1
- new net MCU/PA11: TP1.1
- new net MCU/PA12: TP2.1
Other:
- sheet Connector ports: added SPI_CS, SPI_MISO, SPI_MOSI, SPI_SCK; removed none
- moved on the sheet: D1, D2, R21, R22
