File: can.kicad_sch (KiCad schematic)
At the start: 11 parts, among them SW1 SW_DIP_x02, U3 MCP2562FD-E-SN, U4 MCP2562FD-E-SN

Commit message: fix
Connections:
- net CAN1_L: now also SW1.3; no longer SW1.1
- net CAN2_L: now also SW1.1; no longer SW1.3
- net at R20.2: now also SW1.4; no longer SW1.2
- net at R19.1: now also SW1.2; no longer SW1.4
Other:
- moved on the sheet: SW1
Changed lines of the file:
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@@
 		(shape bidirectional)
 		(at 152.4 68.58 0)
-		(fields_autoplaced yes)
 		(effects
 			(font
@@
 		(shape bidirectional)
 		(at 34.29 110.49 180)
-		(fields_autoplaced yes)
 		(effects
 			(font
@@
 		(shape bidirectional)
 		(at 152.4 110.49 0)
-		(fields_autoplaced yes)
 		(effects
 			(font
@@
 		(shape bidirectional)
 		(at 152.4 115.57 0)
-		(fields_autoplaced yes)
 		(effects
 			(font
@@
 		(shape bidirectional)
 		(at 152.4 63.5 0)
-		(fields_autoplaced yes)
 		(effects
 			(font
@@
 		(shape bidirectional)
 		(at 33.02 60.96 180)
-		(fields_autoplaced yes)
 		(effects
 			(font
@@
 		(shape bidirectional)
 		(at 33.02 63.5 180)
-		(fields_autoplaced yes)
 		(effects
 			(font
@@
 		(shape bidirectional)
 		(at 34.29 107.95 180)
-		(fields_autoplaced yes)
 		(effects
 			(font
@@
 	(symbol
 		(lib_id "Switch:SW_DIP_x02")
-		(at 130.81 91.44 0)
-		(unit 1)
-		(exclude_from_sim no)
-		(in_bom yes)
-		(on_board yes)
-		(dnp no)
-		(fields_autoplaced yes)
+		(at 130.81 88.9 180)
+		(unit 1)
+		(exclude_from_sim no)
+		(in_bom yes)
+		(on_board yes)
+		(dnp no)
 		(property "Reference" "SW1"
-			(at 130.81 81.28 0)
+			(at 130.81 99.06 0)
 			(effects
 				(font
@@
 		)
 		(property "Value" "SW_DIP_x02"
-			(at 130.81 83.82 0)
+			(at 130.81 96.52 0)
 			(effects
 				(font
@@
 		)
 		(property "Footprint" "Button_Switch_SMD:SW_DIP_SPSTx02_Slide_Copal_CHS-02B_W7.62mm_P1.27mm"
-			(at 130.81 91.44 0)
+			(at 130.81 88.9 0)
 			(effects
 				(font
@@
 		)
 		(property "Datasheet" "~"
-			(at 130.81 91.44 0)
+			(at 130.81 88.9 0)
 			(effects
 				(font
@@
 		)
 		(property "Description" "2x DIP Switch, Single Pole Single Throw (SPST) switch, small symbol"
-			(at 130.81 91.44 0)
-			(effects
-				(font
+			(at 130.81 88.9 0)
+			(effects
+				(font
