File: connectro.kicad_sch (KiCad schematic)
At the start: 3 parts, among them J2 ST-Link, J3 Conn_01x10, J4 Conn_01x10

Commit message: fix
Connections:
- net CAN1_H: now also J3.10 (Pin_10); no longer J4.10 (Pin_10)
- net CAN1_L: now also J3.9 (Pin_9); no longer J4.9 (Pin_9)
- net CAN1_RD: now also J3.7 (Pin_7); no longer J4.7 (Pin_7)
- net CAN1_TD: now also J3.8 (Pin_8); no longer J4.8 (Pin_8)
- net CAN2_H: now also J4.10 (Pin_10); no longer J3.10 (Pin_10)
- net CAN2_L: now also J4.9 (Pin_9); no longer J3.9 (Pin_9)
- net CAN2_RD: now also J4.7 (Pin_7); no longer J3.7 (Pin_7)
- net CAN2_TD: now also J4.8 (Pin_8); no longer J3.8 (Pin_8)
- net GND: no longer J3.1 (Pin_1)
- net SPI_MISO: now reaches J3.2 (Pin_2)
- net SPI_SCK: now reaches J3.3 (Pin_3)
- net SPI_CS: now reaches J3.4 (Pin_4)
- new net SPI_MOSI: J3.1 (Pin_1)
- no-connect marks 7 -> 4
Other:
- moved on the sheet: J4
