File: ethernet.kicad_sch (KiCad schematic)
At the start: 33 parts, among them J1 RJ45_Amphenol_RJMG1BD3B8K1ANR, U2 LAN8742A, Y2 25MHz

Commit message: fix
Parts:
- removed J1: RJ45_Amphenol_RJMG1BD3B8K1ANR, Connector_RJ:RJ45_Amphenol_RJMG1BD3B8K1ANR, symbol Connector:RJ45_Amphenol_RJMG1BD3B8K1ANR
- added J5: RJ45_Hanrun_HR911105A_Horizontal, Connector_RJ:RJ45_Hanrun_HR911105A_Horizontal, symbol Connector:RJ45_Hanrun_HR911105A_Horizontal
Connections:
- net LED1: now also J5.12
- net LED2: now also J5.9
- net at C17.1, C18.1, C19.1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: now also J5.4 (TCT), J5.5 (RCT)
- net at R13.2, U2.20 (TXN): now also J5.2 (TD-)
- net at R12.2, U2.21 (TXP): now also J5.1 (TD+)
- net at R15.2, U2.22 (RXN): now also J5.6 (RD-)
- net at R14.2, U2.23 (RXP): now also J5.3 (RD+)
- net at R17.1: now also J5.11
- net at R18.1: now also J5.10
- net at JP1.1 (A): now also J5.8, J5.SH
Other:
- moved on the sheet: R17, R18
Changed lines of the file:
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@@
 	(wire
 		(pts
-			(xy 260.35 76.2) (xy 266.7 76.2)
+			(xy 260.35 78.74) (xy 266.7 78.74)
 		)
 		(stroke
@@
 	(wire
 		(pts
-			(xy 260.35 86.36) (xy 266.7 86.36)
+			(xy 260.35 88.9) (xy 266.7 88.9)
 		)
 		(stroke
@@
 	)
 	(label "LED2"
-		(at 260.35 88.9 0)
-		(fields_autoplaced yes)
+		(at 260.35 86.36 0)
 		(effects
 			(font
@@
 	)
 	(label "LED1"
-		(at 260.35 78.74 0)
-		(fields_autoplaced yes)
+		(at 260.35 76.2 0)
 		(effects
 			(font
@@
 	(label "LED2"
 		(at 184.15 124.46 180)
-		(fields_autoplaced yes)
 		(effects
 			(font
@@
 	(label "LED1"
 		(at 154.94 96.52 0)
-		(fields_autoplaced yes)
 		(effects
 			(font
@@
 	(label "LED2"
 		(at 154.94 99.06 0)
-		(fields_autoplaced yes)
 		(effects
 			(font
@@
 		(shape bidirectional)
 		(at 44.45 99.06 180)
-		(fields_autoplaced yes)
 		(effects
 			(font
@@
 		(shape bidirectional)
 		(at 44.45 73.66 180)
-		(fields_autoplaced yes)
 		(effects
 			(font
@@
 		(shape bidirectional)
 		(at 44.45 93.98 180)
-		(fields_autoplaced yes)
 		(effects
 			(font
@@
 		(shape bidirectional)
 		(at 44.45 81.28 180)
-		(fields_autoplaced yes)
 		(effects
 			(font
@@
 		(shape bidirectional)
 		(at 44.45 101.6 180)
-		(fields_autoplaced yes)
 		(effects
 			(font
@@
 		(shape bidirectional)
 		(at 44.45 76.2 180)
-		(fields_autoplaced yes)
 		(effects
 			(font
@@
 		(shape bidirectional)
 		(at 44.45 91.44 180)
-		(fields_autoplaced yes)
 		(effects
 			(font
@@
 		(shape bidirectional)
 		(at 44.45 83.82 180)
-		(fields_autoplaced yes)
 		(effects
 			(font
@@
 		(shape bidirectional)
 		(at 44.45 88.9 180)
-		(fields_autoplaced yes)
 		(effects
 			(font
@@
 		(shape bidirectional)
 		(at 44.45 78.74 180)
-		(fields_autoplaced yes)
 		(effects
 			(font
@@
 	)
 	(symbol
-		(lib_id "Connector:RJ45_Amphenol_RJMG1BD3B8K1ANR")
-		(at 237.49 83.82 0)
-		(unit 1)
-		(exclude_from_sim no)
-		(in_bom yes)
-		(on_board yes)
-		(dnp no)
-		(fields_autoplaced yes)
-		(property "Reference" "J1"
-			(at 238.76 69.85 0)
-			(effects
-				(font
-					(size 1.27 1.27)
-				)
-			)
-		)
-		(property "Value" "RJ45_Amphenol_RJMG1BD3B8K1ANR"
-			(at 238.76 72.39 0)
-			(effects
-				(font
-					(size 1.27 1.27)
-				)
-			)
-		)
-		(property "Footprint" "Connector_RJ:RJ45_Amphenol_RJMG1BD3B8K1ANR"
-			(at 237.49 71.12 0)
-			(effects
-				(font
-					(size 1.27 1.27)
-				)
-				(hide yes)
-			)
-		)
-		(property "Datasheet" "https://www.amphenol-cs.com/media/wysiwyg/files/drawing/rjmg1bd3b8k1anr.pdf"
-			(at 237.49 68.58 0)
-			(effects
-				(font
-					(size 1.27 1.27)
-				)
-				(hide yes)
-			)
-		)
-		(property "Description" "1 Port RJ45 Magjack Connector Through Hole 10/100 Base-T, AutoMDIX"
-			(at 237.49 83.82 0)
-			(effects
-				(font
-					(size 1.27 1.27)
-				)
-				(hide yes)
-			)
-		)
-		(pin "R2"
-		)
-		(pin "L4"
-		)
-		(pin "L1"
-		)
-		(pin "L2"
-		)
-		(pin "L3"
-		)
-		(pin "R3"
-		)
-		(pin "R7"
-		)
-		(pin "R8"
-		)
-		(pin "SH"
-		)
-		(pin "R1"
-		)
-		(pin "R6"
-		)
-		(pin "R5"
-		)
-		(pin "R4"
-		)
-		(instances
-			(project "CANgatewayE"
-				(path "/7367c43a-3a81-4578-802c-80993d597842/e7499d42-dd47-452d-b831-bf66f386bd66"
-					(reference "J1")
-					(unit 1)
-				)
-			)
-		)
-	)
-	(symbol
 		(lib_id "Device:C_Small")
 		(at 115.57 55.88 0)
@@
 	(symbol
 		(lib_id "power:GND")
-		(at 271.78 76.2 90)
+		(at 271.78 78.74 90)
 		(unit 1)
 		(exclude_from_sim no)
@@
 		(fields_autoplaced yes)
 		(property "Reference" "#PWR026"
-			(at 278.13 76.2 0)
+			(at 278.13 78.74 0)
 			(effects
 				(font
@@
 		)
 		(property "Value" "GND"
-			(at 275.59 76.1999 90)
+			(at 275.59 78.7399 90)
 			(effects
 				(font
@@
 		)
 		(property "Footprint" ""
-			(at 271.78 76.2 0)
+			(at 271.78 78.74 0)
 			(effects
 				(font
@@
 		)
 		(property "Datasheet" ""
-			(at 271.78 76.2 0)
+			(at 271.78 78.74 0)
 			(effects
 				(font
@@
 		)
 		(property "Description" "Power symbol creates a global label with name \"GND\" , ground"
-			(at 271.78 76.2 0)
+			(at 271.78 78.74 0)
 			(effects
 				(font
@@
 	(symbol
 		(lib_id "Device:R_Small")
-		(at 269.24 86.36 90)
+		(at 269.24 88.9 90)
 		(unit 1)
 		(exclude_from_sim no)
@@
 		(fields_autoplaced yes)
 		(property "Reference" "R18"
-			(at 269.24 81.28 90)
+			(at 269.24 83.82 90)
 			(effects
 				(font
@@
 		)
 		(property "Value" "270"
-			(at 269.24 83.82 90)
+			(at 269.24 86.36 90)
 			(effects
 				(font
@@
 		)
 		(property "Footprint" "Resistor_SMD:R_0402_1005Metric"
-			(at 269.24 86.36 0)
+			(at 269.24 88.9 0)
 			(effects
 				(font
@@
 		)
 		(property "Datasheet" "~"
-			(at 269.24 86.36 0)
+			(at 269.24 88.9 0)
 			(effects
 				(font
@@
 		)
 		(property "Description" "Resistor, small symbol"
-			(at 269.24 86.36 0)
+			(at 269.24 88.9 0)
 			(effects
 				(font
@@
 	(symbol
 		(lib_id "power:GND")
-		(at 271.78 86.36 90)
+		(at 271.78 88.9 90)
 		(unit 1)
 		(exclude_from_sim no)
@@
 		(fields_autoplaced yes)
 		(property "Reference" "#PWR027"
-			(at 278.13 86.36 0)
+			(at 278.13 88.9 0)
 			(effects
 				(font
@@
 		)
 		(property "Value" "GND"
-			(at 275.59 86.3599 90)
+			(at 275.59 88.8999 90)
 			(effects
 				(font
@@
 		)
 		(property "Footprint" ""
-			(at 271.78 86.36 0)
+			(at 271.78 88.9 0)
 			(effects
 				(font
@@
 		)
 		(property "Datasheet" ""
-			(at 271.78 86.36 0)
+			(at 271.78 88.9 0)
 			(effects
 				(font
@@
 		)
 		(property "Description" "Power symbol creates a global label with name \"GND\" , ground"
-			(at 271.78 86.36 0)
+			(at 271.78 88.9 0)
 			(effects
 				(font
@@
 	(symbol
 		(lib_id "Device:R_Small")
-		(at 269.24 76.2 90)
+		(at 269.24 78.74 90)
 		(unit 1)
 		(exclude_from_sim no)
@@
 		(fields_autoplaced yes)
 		(property "Reference" "R17"
-			(at 269.24 71.12 90)
+			(at 269.24 73.66 90)
 			(effects
 				(font
@@
 		)
 		(property "Value" "270"
-			(at 269.24 73.66 90)
+			(at 269.24 76.2 90)
 			(effects
 				(font
@@
 		)
 		(property "Footprint" "Resistor_SMD:R_0402_1005Metric"
-			(at 269.24 76.2 0)
+			(at 269.24 78.74 0)
 			(effects
 				(font
@@
 		)
 		(property "Datasheet" "~"
-			(at 269.24 76.2 0)
+			(at 269.24 78.74 0)
 			(effects
 				(font
@@
 		)
 		(property "Description" "Resistor, small symbol"
-			(at 269.24 76.2 0)
+			(at 269.24 78.74 0)
 			(effects
 				(font
@@
 					(unit 1)
 				)
+			)
+		)
+	)
+	(symbol
+		(lib_id "Connector:RJ45_Hanrun_HR911105A_Horizontal")
+		(at 237.49 83.82 0)
+		(unit 1)
+		(exclude_from_sim no)
+		(in_bom yes)
+		(on_board yes)
+		(dnp no)
+		(fields_autoplaced yes)
+		(property "Reference" "J5"
+			(at 238.76 69.85 0)
+			(effects
+				(font
+					(size 1.27 1.27)
+				)
+			)
+		)
+		(property "Value" "RJ45_Hanrun_HR911105A_Horizontal"
+			(at 238.76 72.39 0)
+			(effects
+				(font
+					(size 1.27 1.27)
+				)
+			)
+		)
+		(property "Footprint" "Connector_RJ:RJ45_Hanrun_HR911105A_Horizontal"
+			(at 237.49 71.12 0)
+			(effects
+				(font
+					(size 1.27 1.27)
+				)
+				(hide yes)
+			)
+		)
+		(property "Datasheet" "https://datasheet.lcsc.com/lcsc/1811141815_HANRUN-Zhongshan-HanRun-Elec-HR911105A_C12074.pdf"
+			(at 237.49 68.58 0)
+			(effects
+				(font
+					(size 1.27 1.27)
+				)
+				(hide yes)
+			)
+		)
+		(property "Description" "1 Port RJ45 Magjack Connector Through Hole 10/100 Base-T, AutoMDIX"
+			(at 237.49 83.82 0)
+			(effects
+				(font
+					(size 1.27 1.27)
+				)
+				(hide yes)
+			)
+		)
+		(pin "1"
+		)
+		(pin "11"
+		)
+		(pin "5"
+		)
+		(pin "10"
+		)
+		(pin "3"
+		)
+		(pin "9"
+		)
+		(pin "2"
+		)
+		(pin "12"
+		)
+		(pin "7"
+		)
+		(pin "8"
+		)
+		(pin "4"
+		)
+		(pin "6"
+		)
+		(pin "SH"
+		)
+		(instances
+			(project ""
+				(path "/7367c43a-3a81-4578-802c-80993d597842/e7499d42-dd47-452d-b831-bf66f386bd66"
+					(reference "J5")
+					(unit 1)
+				)
